File: BSBB.kicad_pcb (KiCad board)
At the start: 2 copper layers, 100 x 55 mm, 37 parts, among them J2 Serial Debug, J3 PSU, J4 8P8C_LED_Shielded_x2, J5 XBOX, J6 ModXo I^{2}C, Q1 MMBT4401, Q2 MMBT4401, U1 Teensy4.1, U2 LM1117DT-3.3, U3 MAX3485, U5 PCA9615DP

Commit message: Added top GND fill
Routing:
- net GND: track 39.1 -> 33.6 mm, vias 9 -> 4
- net /Switches.LED: track 33.5 -> 35.3 mm
- net /DMX_RX: track 14.8 -> 15.5 mm
- net /Switches.W0: track 55.5 -> 56.0 mm
- net /Switches.W2: track 45.2 -> 45.7 mm
- net /Switches.W1: track 50.0 -> 50.5 mm
- added copper zone on F.Cu, net GND

Commit message: Small tweaks
Parts:
- R6, R7: value 4.7KΩ -> 2.2KΩ
- moved C1 13.4 mm to (250.8, 83.0), turned to 180 degrees
- moved C6 5.30 mm to (242.0, 92.8), turned to 180 degrees
- moved R1 4.72 mm to (194.8, 78.0), turned to -90 degrees
- moved R2 4.67 mm to (179.0, 78.0), turned to -90 degrees
- moved C2 2.69 mm to (242.0, 94.5), turned to 180 degrees
- moved R5 2.41 mm to (246.5, 83.0), turned to 180 degrees
- moved C3 0.10 mm to (175.7, 78.0)
Routing:
- net /Power/+3.3VSB: track 78.4 -> 67.1 mm
- net GND: track 33.6 -> 25.3 mm, vias 4 -> 12
- net /Switches.LED: track 35.3 -> 27.7 mm
- net /DMX-: track 19.9 -> 23.2 mm
- net /Power/XBOX_PWR_OK: track 10.1 -> 7.05 mm
- net Net-(Q2-B): track 2.08 -> 4.78 mm
- net /Cockpit RJ45 Led: track 30.1 -> 27.7 mm
- net Net-(J4-Pad24): track 5.30 -> 7.74 mm
- net Net-(J4-Pad12): track 5.27 -> 7.65 mm
- net /Power/+5VSB: track 82.3 -> 80.2 mm
- net +12V: track 120.9 -> 118.9 mm
- net /Power/+3.3V: track 104.5 -> 103.8 mm
- net /DMX_~{R}T: track 18.8 -> 19.4 mm

Commit message: Plated pads
Parts:
- H2, H3: footprint MountingHole:MountingHole_4.3mm_M4 -> MountingHole:MountingHole_4.3mm_M4_Pad
- H4: footprint MountingHole:MountingHole_4.3mm_M4 -> MountingHole:MountingHole_4.3mm_M4_ISO7380_Pad
Routing:
- net +5V: track 154.0 -> 136.9 mm
- net +3.3V: track 35.6 -> 36.5 mm
- net /Power/+3.3V: vias 1 -> 0
