File: BSBB.kicad_sch (KiCad schematic)
At the start: 20 parts, among them J2 Serial Debug, J4 8P8C_LED_Shielded_x2, J6 ModXo I^{2}C, U1 Teensy4.1, U3 MAX3485, U5 PCA9615DP

Commit message: Added LCSC part numbers
Parts:
- C3, C5: LCSC (none) -> C6119867
- R1, R2, R8, R9: LCSC (none) -> C2906988
- R6, R7: LCSC (none) -> C2907166
- RN1: LCSC (none) -> C48580704
- U3: LCSC (none) -> C668204
- U5: LCSC (none) -> C3824272
Changed lines of the file:
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@@
 			)
 		)
+		(property "LCSC" ""
+			(at 16.51 22.86 0)
+			(hide yes)
+			(show_name no)
+			(do_not_autoplace no)
+			(effects
+				(font
+					(size 1.27 1.27)
+				)
+			)
+		)
 		(instances
 			(project "BSBB"
@@
 			)
 		)
+		(property "LCSC" "C6119867"
+			(at 219.71 17.78 90)
+			(hide yes)
+			(show_name no)
+			(do_not_autoplace no)
+			(effects
+				(font
+					(size 1.27 1.27)
+				)
+			)
+		)
 		(pin "2"
 		)
@@
 			)
 		)
+		(property "LCSC" "C6119867"
+			(at 208.28 97.79 90)
+			(hide yes)
+			(show_name no)
+			(do_not_autoplace no)
+			(effects
+				(font
+					(size 1.27 1.27)
+				)
+			)
+		)
 		(pin "2"
 		)
@@
 			)
 		)
+		(property "LCSC" ""
+			(at 16.51 29.21 0)
+			(hide yes)
+			(show_name no)
+			(do_not_autoplace no)
+			(effects
+				(font
+					(size 1.27 1.27)
+				)
+			)
+		)
 		(instances
 			(project "BSBB"
@@
 			)
 		)
+		(property "LCSC" ""
+			(at 16.5099 35.6278 0)
+			(hide yes)
+			(show_name no)
+			(do_not_autoplace no)
+			(effects
+				(font
+					(size 1.27 1.27)
+				)
+			)
+		)
 		(instances
 			(project "BSBB"
@@
 			)
 		)
+		(property "LCSC" "C3824272"
+			(at 220.98 49.53 0)
+			(hide yes)
+			(show_name no)
+			(do_not_autoplace no)
+			(effects
+				(font
+					(size 1.27 1.27)
+				)
+			)
+		)
 		(pin "1"
 		)
@@
 			)
 		)
+		(property "LCSC" ""
+			(at 245.11 144.78 0)
+			(hide yes)
+			(show_name no)
+			(do_not_autoplace no)
+			(effects
+				(font
+					(size 1.27 1.27)
+				)
+			)
+		)
 		(pin "16"
 		)
@@
 			)
 		)
+		(property "LCSC" ""
+			(at 251.46 124.46 0)
+			(hide yes)
+			(show_name no)
+			(do_not_autoplace no)
+			(effects
+				(font
+					(size 1.27 1.27)
+				)
+			)
+		)
 		(pin "1"
 		)
@@
 			)
 		)
+		(property "LCSC" "C2906988"
+			(at 237.49 20.32 0)
+			(hide yes)
+			(show_name no)
+			(do_not_autoplace no)
+			(effects
+				(font
+					(size 1.27 1.27)
+				)
+			)
+		)
 		(pin "2"
 		)
@@
 			)
 		)
+		(property "LCSC" "C48580704"
+			(at 247.65 27.94 90)
+			(hide yes)
+			(show_name no)
+			(do_not_autoplace no)
+			(effects
+				(font
+					(size 1.27 1.27)
+				)
+			)
+		)
 		(pin "4"
 		)
@@
 			)
 		)
+		(property "LCSC" "C2906988"
+			(at 270.51 50.8 0)
+			(hide yes)
+			(show_name no)
+			(do_not_autoplace no)
+			(effects
+				(font
+					(size 1.27 1.27)
+				)
+			)
+		)
 		(pin "2"
 		)
@@
 			)
 		)
+		(property "LCSC" ""
+			(at 140.97 105.41 0)
+			(hide yes)
+			(show_name no)
+			(do_not_autoplace no)
+			(effects
+				(font
+					(size 1.27 1.27)
+				)
+			)
+		)
 		(pin "52"
 		)
@@
 			)
 		)
-		(property "Datasheet" ""
+		(property "Datasheet" "C6119867"
 			(at 204.47 21.59 0)
 			(hide yes)
@@
 			)
 		)
+		(property "LCSC" ""
+			(at 204.47 21.59 90)
+			(hide yes)
+			(show_name no)
+			(do_not_autoplace no)
+			(effects
+				(font
+					(size 1.27 1.27)
+				)
+			)
+		)
 		(pin "2"
 		)
@@
 			)
 		)
+		(property "LCSC" "C2906988"
+			(at 237.49 33.02 0)
+			(hide yes)
+			(show_name no)
+			(do_not_autoplace no)
+			(effects
+				(font
+					(size 1.27 1.27)
+				)
+			)
+		)
 		(pin "2"
 		)
@@
 			)
 		)
+		(property "LCSC" "C2907166"
+			(at 198.12 43.18 0)
+			(hide yes)
+			(show_name no)
+			(do_not_autoplace no)
+			(effects
+				(font
+					(size 1.27 1.27)
+				)
+			)
+		)
 		(pin "2"
 		)
@@
 			)
 		)
+		(property "LCSC" "C668204"
+			(at 220.98 82.55 0)
+			(hide yes)
+			(show_name no)
+			(do_not_autoplace no)
+			(effects
+				(font
+					(size 1.27 1.27)
+				)
+			)
+		)
 		(pin "3"
 		)
@@
 			)
 		)
+		(property "LCSC" "C2907166"
+			(at 205.74 43.18 0)
+			(hide yes)
+			(show_name no)
+			(do_not_autoplace no)
+			(effects
+				(font
+					(size 1.27 1.27)
+				)
+			)
+		)
 		(pin "2"
 		)
@@
 			)
 		)
+		(property "LCSC" ""
+			(at 16.51 16.51 0)
+			(hide yes)
+			(show_name no)
+			(do_not_autoplace no)
+			(effects
+				(font
+					(size 1.27 1.27)
+				)
+			)
+		)
 		(instances
 			(project "BSBB"
@@
 			)
 		)
+		(property "LCSC" ""
+			(at 259.08 62.23 0)
+			(hide yes)
+			(show_name no)
+			(do_not_autoplace no)
+			(effects
+				(font
+					(size 1.27 1.27)
+				)
+			)
+		)
 		(pin "16"
 		)
@@
 			)
 		)
+		(property "LCSC" "C2906988"
+			(at 256.54 133.35 0)
+			(hide yes)
+			(show_name no)
+			(do_not_autoplace no)
+			(effects
+				(font
+					(size 1.27 1.27)
+				)
+			)
+		)
 		(pin "2"
 		)
@@
 			(at 251.46 114.3 0)
 			(hide yes)
+			(show_name no)
+			(do_not_autoplace no)
+			(effects
+				(font
+					(size 1.27 1.27)
+				)
+			)
+		)
+		(property "LCSC" ""
+			(at 251.46 114.3 0)
+			(hide yes)

Commit message: Small tweaks
Parts:
- R6, R7: value 4.7KΩ -> 2.2KΩ; LCSC C2907166 -> C2907005
Changed lines of the file:
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@@
 			)
 		)
-		(property "Value" "4.7KΩ"
+		(property "Value" "2.2KΩ"
 			(at 194.056 40.64 0)
 			(show_name no)
@@
 			)
 		)
-		(property "LCSC" "C2907166"
+		(property "LCSC" "C2907005"
 			(at 198.12 43.18 0)
 			(hide yes)
@@
 			)
 		)
-		(property "Value" "4.7KΩ"
+		(property "Value" "2.2KΩ"
 			(at 201.93 40.386 0)
 			(show_name no)
@@
 			)
 		)
-		(property "LCSC" "C2907166"
+		(property "LCSC" "C2907005"
 			(at 205.74 43.18 0)
 			(hide yes)

Commit message: Plated pads
Parts:
- H2, H3: footprint MountingHole:MountingHole_4.3mm_M4 -> MountingHole:MountingHole_4.3mm_M4_Pad; symbol Mechanical:MountingHole -> Mechanical:MountingHole_Pad
- H4: footprint MountingHole:MountingHole_4.3mm_M4 -> MountingHole:MountingHole_4.3mm_M4_ISO7380_Pad; symbol Mechanical:MountingHole -> Mechanical:MountingHole_Pad
Connections:
- net GND: now also H2.1, H3.1, H4.1
Other:
- moved on the sheet: C3, C4, C5, H1
